File: hardware/top_connector/top_connector.kicad_pcb (KiCad board)
At the start: 2 copper layers, 38.5 x 28.5 mm, 14 parts, among them J1 to prev top connector, J2 to next top connector, J3 to module, U1 XL1509-5.0, U2 74LVC1G66

Commit message: Switching to KiCad: Added side panel schematic and board
Other:
- board text added: "${TITLE}"
- board text removed: "${PROJECTNAME}"
Changed lines of the file:
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@@
 		(title "Top Connector")
 		(date "2024-07-26")
-		(rev "2.0.0")
+		(rev "2.0.1")
 		(company "OpenFlap")
 		(comment 1 "Designer: Toon Van Eyck")
@@
 			)
 		)
-		(model "${KICAD8_3DMODEL_DIR}/Connector_Samtec_HLE_SMD.3dshapes/Samtec_HLE-108-02-xxx-DV_2x08_P2.54mm_Horizontal.wrl"
+		(model "${KIPRJMOD}/../resources/HLE-108-02-L-DV-BE-TR.stp"
 			(offset
-				(xyz 0 0 0)
-			)
-			(scale
-				(xyz 1 1 1)
-			)
-			(rotate
-				(xyz 0 0 0)
-			)
-		)
-		(model "${KIPRJMOD}/HLE-108-02-L-DV-BE-TR.stp"
-			(offset
-				(xyz 0 0 0.15)
+				(xyz 0 0 0.1)
 			)
 			(scale
@@
 			)
 			(rotate
-				(xyz -90 0 -180)
+				(xyz -90 0 0)
 			)
 		)
@@
 			(justify left bottom mirror)
 		)
-		(render_cache "2.0.0" 90
+		(render_cache "2.0.1" 90
 			(polygon
 				(pts
@@
 			(polygon
 				(pts
-					(xy 123.569319 131.862025) (xy 123.625877 131.864201) (xy 123.679481 131.869639) (xy 123.73013 131.87834)
-					(xy 123.777826 131.890304) (xy 123.829739 131.908386) (xy 123.836802 131.911321) (xy 123.883411 131.933818)
-					(xy 123.930611 131.963707) (xy 123.971338 131.998054) (xy 124.005593 132.036858) (xy 124.032628 132.079478)
-					(xy 124.051938 132.12503) (xy 124.063525 132.173512) (xy 124.067387 132.224925) (xy 124.063525 132.276918)
-					(xy 124.051938 132.325675) (xy 124.032628 132.371196) (xy 124.005593 132.41348) (xy 123.997636 132.42354)
-					(xy 123.961763 132.461031) (xy 123.919418 132.494126) (xy 123.877056 132.519478) (xy 123.829739 132.541464)
-					(xy 123.822569 132.544319) (xy 123.770082 132.561766) (xy 123.721894 132.573187) (xy 123.670752 132.581344)
-					(xy 123.616656 132.586238) (xy 123.559606 132.58787) (xy 123.549803 132.587824) (xy 123.492811 132.585649)
-					(xy 123.438944 132.580211) (xy 123.388202 132.57151) (xy 123.340586 132.559546) (xy 123.288985 132.541464)
-					(xy 123.281952 132.538529) (xy 123.235541 132.516062) (xy 123.18854 132.486265) (xy 123.14798 132.452071)
-					(xy 123.123795 132.424715) (xy 123.274086 132.424715) (xy 123.305681 132.439568) (xy 123.352495 132.456427)
-					(xy 123.400115 132.468923) (xy 123.404648 132.46993) (xy 123.456432 132.478895) (xy 123.506564 132.48369)
-					(xy 123.559606 132.485288) (xy 123.57535 132.485162) (xy 123.628381 132.482737) (xy 123.678186 132.477228)
-					(xy 123.731156 132.467153) (xy 123.779913 132.453048) (xy 123.796996 132.446771) (xy 123.843866 132.425158)
-					(xy 123.88824 132.39625) (xy 123.924505 132.362189) (xy 123.951682 132.323597) (xy 123.96995 132.276628)
-					(xy 123.97604 132.224925) (xy 123.971222 132.178466) (xy 123.954792 132.131825) (xy 123.926703 132.089859)
-					(xy 123.274086 132.424715) (xy 123.123795 132.424715) (xy 123.113863 132.41348) (xy 123.086721 132.371196)
-					(xy 123.067334 132.325675) (xy 123.055702 132.276918) (xy 123.051825 132.224925) (xy 123.143172 132.224925)
-					(xy 123.14799 132.271383) (xy 123.16442 132.318025) (xy 123.192509 132.359991) (xy 123.845126 132.025134)
-					(xy 123.813551 132.010262) (xy 123.766822 131.993318) (xy 123.719341 131.980682) (xy 123.714793 131.97969)
-					(xy 123.662875 131.970859) (xy 123.612671 131.966136) (xy 123.559606 131.964562) (xy 123.54392 131.964688)
-					(xy 123.491048 131.967112) (xy 123.441331 131.972622) (xy 123.388376 131.982697) (xy 123.339543 131.996802)
-					(xy 123.322375 132.003123) (xy 123.275326 132.02484) (xy 123.23089 132.05382) (xy 123.194707 132.087905)
-					(xy 123.16753 132.126473) (xy 123.149261 132.173361) (xy 123.143172 132.224925) (xy 123.051825 132.224925)
-					(xy 123.055702 132.173512) (xy 123.067334 132.12503) (xy 123.086721 132.079478) (xy 123.113863 132.036858)
-					(xy 123.121788 132.026739) (xy 123.157516 131.989049) (xy 123.199686 131.955817) (xy 123.24187 131.930395)
-					(xy 123.288985 131.908386) (xy 123.296096 131.905531) (xy 123.348305 131.888083) (xy 123.396442 131.876663)
-					(xy 123.447705 131.868506) (xy 123.502092 131.863611) (xy 123.559606 131.86198)
+					(xy 124.052 131.921087) (xy 123.963339 131.921087) (xy 123.963339 132.16997) (xy 123.176877 132.16997)
+					(xy 123.286787 131.921087) (xy 123.19373 131.921087) (xy 123.067212 132.208072) (xy 123.067212 132.271331)
+					(xy 123.963339 132.271331) (xy 123.963339 132.55563) (xy 124.052 132.55563)
 				)
 			)
@@
 		)
 	)
-	(gr_text "${PROJECTNAME}\n"
+	(gr_text "${TITLE}\n"
 		(at 120.666 130.986 90)
 		(layer "B.SilkS")
