File: hardware/module/side_panel/side_panel.kicad_pcb (KiCad board)
At the start: 2 copper layers, 96 x 120.2 mm, 46 parts, among them J1 Top Connector, J2 Bottom Connecor, J3 Conn_01x05, J7 Conn_01x09, M1 GA12-N20 12V 100rpm, Q1 AP2302B, U1 QRE1113GR, U2 QRE1113GR, U3 QRE1113GR, U4 QRE1113GR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

Commit message: fix erc & drc for sidepanel
Parts:
- removed TP3: TestPoint, Connector_PinHeader_1.27mm:PinHeader_1x01_P1.27mm_Vertical
- renumbered REF** to OSHW-LOGO-1, REF** to OSHW-LOGO-2
