File: hardware/top_connector/src/top_connector.kicad_pcb (KiCad board)
At the start: 2 copper layers, 38.5 x 28.5 mm, 14 parts, among them J1 to prev top connector, J2 to next top connector, J3 to module, U1 XL1509-5.0, U2 74LVC1G66

Commit message: Use kibot on sidepanel and top connector
Parts:
- renumbered REF** to OSHW_LOGO_1
