File: hardware/top_connector/src/top_connector.kicad_pcb (KiCad board)
At the start: 2 copper layers, 57.9 x 30.7 mm, 15 parts, among them J1 Conn_02x09_Odd_Even, J2 Conn_02x09_Odd_Even, J3 Conn_02x07_Odd_Even, U1 XL1509-5.0, U2 74LVC1G66

Commit message: Add test points to pcb's
Parts:
- added TP1: TestPoint, TestPoint:TestPoint_Pad_D1.5mm, B.Cu at (115.7, 146.2)
- C4: value 22uF -> 220uF; footprint Capacitor_SMD:CP_Elec_5x5.4 -> Capacitor_SMD:CP_Elec_6.3x7.7
- moved D3 20.0 mm to (122.7, 135.4), turned to -90 degrees
- moved D2 10.7 mm to (98.5, 146.0), turned to 180 degrees
- moved C4 1.18 mm to (116.2, 134.7)
Routing:
- net Net-(D1-K): track 21.9 -> 12.2 mm, vias 3 -> 0
- net GND: track 19.4 -> 24.3 mm
- net +5V: track 62.6 -> 60.9 mm, vias 0 -> 1
- net +12V: track 46.0 -> 45.0 mm
